Commit message: Fitted slambot with laser sensor

File: urdf/slambot.urdf.xacro (robot description, xacro)
@@ -8,4 +8,7 @@
 <xacro:property name = "base_height" value = "0.05" />
 <xacro:property name = "base_mass" value = "100.0" />
+<xacro:property name = "laser_mass" value = "0.1" />
+<xacro:property name = "laser_height" value = "0.1" />
+<xacro:property name = "laser_radius" value = "0.1" />
 	<link name = "base_link" >
 		<inertial>
@@ -32,4 +35,28 @@
 		</collision>
 	</link>
+	<link name = "laser_link" >
+		<inertial>
+			<mass value = "${laser_mass}" />
+			<origin xyz = "0 0 0" rpy = "0 0 0" />
+			<inertia ixx = "0.0"
+					 ixy = "0.0"
+					 ixz = "0.0"
+					 iyy = "0.0"
+					 iyz = "0.0"
+					 izz = "0.0" />
+		</inertial>
+		<visual name = "laser_link_visual" >
+			<origin xyz = "0 0 0" rpy = "0 0 0" />
+			<geometry>
+				<cylinder length = "${laser_height}" radius = "${laser_radius}" />
+			</geometry>
+		</visual>
+		<collision name = "laser_link_collision" >
+			<origin xyz = "0 0 0" rpy = "0 0 0" />
+			<geometry>
+				<cylinder length = "${laser_height}" radius = "${laser_radius}" />
+			</geometry>
+		</collision>
+	</link>
 	<link name = "front_right_wheel_link" >
 		<inertial>
@@ -128,4 +155,11 @@
 		</collision>
 	</link>
+	<joint name = "laser_joint" type = "revolute" >
+		<parent link = "base_link" />
+		<child link = "laser_link" />
+		<origin xyz = "0 ${base_length/2-laser_radius} ${wheel_radius+laser_height/2+base_height/2}" rpy = "0 0 0" />
+		<axis xyz = "0 0 1" />
+		<limit lower = "0.0" upper = "0.0" velocity = "0.0" effort = "0.0" />
+	</joint>
 	<joint name = "front_right_wheel_joint" type = "continuous" >
 		<parent link = "base_link" />
@@ -193,8 +227,39 @@
     </transmission>
 	<gazebo>
-	  <static> false </static>
-	  <plugin name="gazebo_ros_control" filename="libgazebo_ros_control.so">
-	    <robotNamespace> /slambot </robotNamespace>
-	  </plugin>
+		<static> false </static>
+		<plugin name="gazebo_ros_control" filename="libgazebo_ros_control.so">
+			<robotNamespace> /slambot </robotNamespace>
+		</plugin>
 	</gazebo>
+	<gazebo reference = "laser_link">
+		<sensor type="ray" name="laser">
+			<pose>0 0 ${laser_height/2+0.01} 0 0 1.571</pose>
+			<visualize>true</visualize>
+			<update_rate>40</update_rate>
+			<ray>
+		    	<scan>
+		      		<horizontal>
+		        		<samples>720</samples>
+		        		<resolution>1</resolution>
+		        		<min_angle>-1.570796</min_angle>
+		        		<max_angle>1.570796</max_angle>
+		      		</horizontal>
+		    	</scan>
+		    	<range>
+		      		<min>0.10</min>
+		      		<max>30.0</max>
+		      		<resolution>0.01</resolution>
+		    	</range>
+		    	<noise>
+		      		<type>gaussian</type>
+		      		<mean>0.0</mean>
+		      		<stddev>0.01</stddev>
+		    	</noise>
+		  	</ray>
+			<plugin name="gazebo_ros_head_hokuyo_controller" filename="libgazebo_ros_laser.so">
+				<topicName>/scan</topicName>
+				<frameName>base_link</frameName>
+			</plugin>
+		</sensor>
+  	</gazebo>
 </robot>

Commit message: Stopped visualizing laser

File: urdf/slambot.urdf.xacro (robot description, xacro)
@@ -3,9 +3,9 @@
 <xacro:property name = "wheel_radius" value = "0.1" />
 <xacro:property name = "wheel_width" value = "0.075" />
-<xacro:property name = "wheel_mass" value = "0.1" />
+<xacro:property name = "wheel_mass" value = "10.0" />
 <xacro:property name = "base_width" value = "0.4" />
 <xacro:property name = "base_length" value = "0.5" />
 <xacro:property name = "base_height" value = "0.05" />
-<xacro:property name = "base_mass" value = "100.0" />
+<xacro:property name = "base_mass" value = "10000.0" />
 <xacro:property name = "laser_mass" value = "0.1" />
 <xacro:property name = "laser_height" value = "0.1" />
@@ -166,5 +166,5 @@
 		<child link = "front_right_wheel_link" />
 		<origin xyz = "${base_width/2+wheel_width/2} ${base_length/2-wheel_radius} ${wheel_radius}" rpy = "0 0 0" />
-		<axis xyz = "1 0 0" />
+		<axis xyz = "-1 0 0" />
 	</joint>
 	<joint name = "front_left_wheel_joint" type = "continuous" >
@@ -172,5 +172,5 @@
 		<child link = "front_left_wheel_link" />
 		<origin xyz = "-${base_width/2+wheel_width/2} ${base_length/2-wheel_radius} ${wheel_radius}" rpy = "0 0 0" />
-		<axis xyz = "1 0 0" />
+		<axis xyz = "-1 0 0" />
 	</joint>
 	<joint name = "back_right_wheel_joint" type = "continuous" >
@@ -178,5 +178,5 @@
 		<child link = "back_right_wheel_link" />
 		<origin xyz = "${base_width/2+wheel_width/2} -${base_length/2-wheel_radius} ${wheel_radius}" rpy = "0 0 0" />
-		<axis xyz = "1 0 0" />
+		<axis xyz = "-1 0 0" />
 	</joint>
 	<joint name = "back_left_wheel_joint" type = "continuous" >
@@ -184,5 +184,5 @@
 		<child link = "back_left_wheel_link" />
 		<origin xyz = "-${base_width/2+wheel_width/2} -${base_length/2-wheel_radius} ${wheel_radius}" rpy = "0 0 0" />
-		<axis xyz = "1 0 0" />
+		<axis xyz = "-1 0 0" />
 	</joint>
 	<transmission name = "front_right_wheel_motor" >
@@ -234,7 +234,7 @@
 	<gazebo reference = "laser_link">
 		<sensor type="ray" name="laser">
-			<pose>0 0 ${laser_height/2+0.01} 0 0 1.571</pose>
-			<visualize>true</visualize>
-			<update_rate>40</update_rate>
+			<pose> 0 0.01 ${laser_height/2} 0 0 1.571 </pose>
+			<visualize> false </visualize>
+			<update_rate> 40 </update_rate>
 			<ray>
 		    	<scan>
@@ -258,6 +258,6 @@
 		  	</ray>
 			<plugin name="gazebo_ros_head_hokuyo_controller" filename="libgazebo_ros_laser.so">
-				<topicName>/scan</topicName>
-				<frameName>base_link</frameName>
+				<topicName> /scan </topicName>
+				<frameName> base_link </frameName>
 			</plugin>
 		</sensor>

Commit message: Laser scan in base frame for now, will update to laser frame with appropriate tf transformation

File: urdf/slambot.urdf.xacro (robot description, xacro)
@@ -35,5 +35,5 @@
 		</collision>
 	</link>
-	<link name = "laser_link" >
+	<!--link name = "laser_link" >
 		<inertial>
 			<mass value = "${laser_mass}" />
@@ -58,5 +58,5 @@
 			</geometry>
 		</collision>
-	</link>
+	</link-->
 	<link name = "front_right_wheel_link" >
 		<inertial>
@@ -155,5 +155,5 @@
 		</collision>
 	</link>
-	<joint name = "laser_joint" type = "revolute" >
+	<!--joint name = "laser_joint" type = "revolute" >
 		<parent link = "base_link" />
 		<child link = "laser_link" />
@@ -161,5 +161,5 @@
 		<axis xyz = "0 0 1" />
 		<limit lower = "0.0" upper = "0.0" velocity = "0.0" effort = "0.0" />
-	</joint>
+	</joint-->
 	<joint name = "front_right_wheel_joint" type = "continuous" >
 		<parent link = "base_link" />
@@ -232,7 +232,8 @@
 		</plugin>
 	</gazebo>
-	<gazebo reference = "laser_link">
+	<gazebo reference = "base_link">
 		<sensor type="ray" name="laser">
-			<pose> 0 0.01 ${laser_height/2} 0 0 1.571 </pose>
+			<!--pose> 0 0.01 ${laser_height/2} 0 0 1.571 </pose-->
+			<pose> 0 0 ${2.5*laser_height} 0 0 1.571 </pose>
 			<visualize> false </visualize>
 			<update_rate> 40 </update_rate>

Commit message: Increased laser scan range

File: urdf/slambot.urdf.xacro (robot description, xacro)
@@ -243,6 +243,6 @@
 		        		<samples>720</samples>
 		        		<resolution>1</resolution>
-		        		<min_angle>-1.570796</min_angle>
-		        		<max_angle>1.570796</max_angle>
+		        		<min_angle>-${pi}</min_angle>
+		        		<max_angle>${pi}</max_angle>
 		      		</horizontal>
 		    	</scan>
@@ -263,4 +263,5 @@
 			</plugin>
 		</sensor>
+		<material> Gazebo/Orange </material>
   	</gazebo>
 </robot>
